File: hardware/kicad/hierarchical_sheets/kx134-1211.kicad_sch (KiCad schematic)
At the start: 0 parts

Commit message: finished KX134
Parts:
- added C6, C7: 100n, symbol Device:C
- added U4: KX134-1211, Package_LGA:LGA-12_2x2mm_P0.5mm, symbol Sensor_Motion:KX122-1042
Connections:
- new net +3.3V: C6.1, C7.1, U4.3 (IO_VDD), U4.7 (VDD)
- new net GND: C6.2, C7.2, U4.8 (GND), U4.9 (GND)
- new net MISO: U4.1 (SDO/ADDR)
- new net MOSI: U4.2 (SDI/SDA)
- new net SCK: U4.12 (SCLK/SCL)
- new net ~{CS}: U4.10 (~{nCS})
- no-connect marks 0 -> 4
